File: ControlBoard/ControlBoard.kicad_sch (KiCad schematic)
At the start: 14 parts

Commit message: Use JYC Design
Parts:
- removed C? (x3): 22u, Capacitor_SMD:C_1206_3216Metric_Pad1.33x1.80mm_HandSolder, symbol Device:C
- removed C?: 3.9nf, Capacitor_SMD:C_0603_1608Metric, symbol Device:C
- removed C?: 100n, Capacitor_SMD:C_0603_1608Metric, symbol Device:C
- removed C?: 2.2u, Capacitor_SMD:C_1206_3216Metric_Pad1.33x1.80mm_HandSolder, symbol Device:C
- removed C?: DNF, Capacitor_SMD:C_0603_1608Metric, symbol Device:C
- removed C?: 15n, Capacitor_SMD:C_0603_1608Metric, symbol Device:C
- removed C?: 470n, Capacitor_SMD:C_0603_1608Metric, symbol Device:C
- removed R?: 309k, Resistor_SMD:R_0603_1608Metric, symbol Device:R
- removed R?: 909k, Resistor_SMD:R_0603_1608Metric, symbol Device:R
- removed R?: 2.1k, Resistor_SMD:R_0603_1608Metric, symbol Device:R
- removed R?: 10k, Resistor_SMD:R_0603_1608Metric, symbol Device:R
- removed U?: LM3150MH, Package_SO:HTSSOP-14-1EP_4.4x5mm_P0.65mm_EP3.4x5mm_Mask3x3.1mm, symbol 0_RM2023:LM3150MH
- added C1: 100n, Capacitor_SMD:C_0603_1608Metric, symbol Device:C
- added C2: 15n, Capacitor_SMD:C_0603_1608Metric, symbol Device:C
- added C3: 2.2u, Capacitor_SMD:C_0603_1608Metric, symbol Device:C
- added C4: 22u, Capacitor_SMD:C_0603_1608Metric, symbol Device:C
- added C5: 470n, Capacitor_SMD:C_0603_1608Metric, symbol Device:C
- added C7: 3.9nf, Capacitor_SMD:C_0603_1608Metric, symbol Device:C
- added C8: 390pf, Capacitor_SMD:C_0603_1608Metric, symbol Device:C
- added C9: ~, Capacitor_SMD:C_0603_1608Metric, symbol Device:C
- added D1: D_Schottky, Diode_SMD:D_SMF, symbol Device:D_Schottky
- added D3: LED, LED_SMD:LED_0603_1608Metric, symbol Device:LED
- added J1, J2, J3, J4: Conn_02x02_Odd_Even, 0_RM2023:conn_2x02_2.54, symbol Connector_Generic:Conn_02x02_Odd_Even
- added R1: 909k, Resistor_SMD:R_0603_1608Metric, symbol Device:R
- added R2: 2.1k, Resistor_SMD:R_0603_1608Metric, symbol Device:R
- added R5: 8.06M, Resistor_SMD:R_0603_1608Metric, symbol Device:R
- added R7: 309k, Resistor_SMD:R_0603_1608Metric, symbol Device:R
- added R8: 10k, Resistor_SMD:R_0603_1608Metric, symbol Device:R
- added R9: 300k, Resistor_SMD:R_0603_1608Metric, symbol Device:R
- added U1: LM3150MH, Package_SO:HTSSOP-14-1EP_4.4x5mm_P0.65mm_EP3.4x5mm_Mask3x3.1mm, symbol 0_RM2023:LM3150MH
Connections:
- net +24V: now also C1.1, C4.1, J1.1 (Pin_1), R1.2, U1.2 (VIN)
- net BST: now also C5.2, D1.1 (K), U1.12 (BST)
- net FB: now also C7.1, C9.1, R7.1, R8.2, U1.4 (FB)
- net GND: now also C1.2, C2.1, C3.1, C4.2, D3.1 (K), J2.1 (Pin_1), J2.2 (Pin_2), J2.3 (Pin_3), J2.4 (Pin_4), J3.1 (Pin_1), J3.2 (Pin_2), J3.3 (Pin_3), J3.4 (Pin_4), R8.1, U1.14 (PGND), U1.15 (EPAD), U1.5 (SGND_2), U1.9 (SGND)
- net SW: now also C5.1, J1.2 (Pin_2), R2.2, R5.1, U1.10 (SW)
- net VOUT: now also C8.2, C9.2, J4.1 (Pin_1), J4.2 (Pin_2), J4.3 (Pin_3), J4.4 (Pin_4), R7.2, R9.1
- new net: D3.2 (A), R9.2
- new net: C2.2, U1.6 (SS)
- new net: R1.1, U1.7 (RON)
- new net: C7.2, C8.1, R5.2
- new net HG: J1.4 (Pin_4), U1.11 (HG)
- new net ILIM: R2.1, U1.8 (ILIM)
- new net LG: J1.3 (Pin_3), U1.13 (LG)
- new net VCC: C3.2, D1.2 (A), U1.1 (VCC)
