File: 24TO19_JYC_RM2023_V0.4_RY.kicad_sch (KiCad schematic)
At the start: 39 parts, among them J1 Conn_01x02, Q1 BSC070N10NS5, Q2 BSC070N10NS5, U1 LM3150MH

Commit message: decoration location adjustment build
Parts:
- D1, D2: footprint Diode_SMD:D_SMB -> Diode_SMD:D_SMC
