File: 24TO19_JYC_RM2023_V0.41_RY.kicad_sch (KiCad schematic)
At the start: 39 parts, among them J1 Conn_01x02, Q1 BSC070N10NS5, Q2 BSC070N10NS5, U1 LM3150MH

Commit message: Updating to ver 0.41: Changed Caps to THT; Decreased total area. Layout done. Routing pending.
Parts:
- C10, C12, C13, C9: value 100uF -> 22uF
- C11, C4: value 100uF -> 330uF; footprint Capacitor_SMD:CP_Elec_10x10.5 -> Capacitor_THT:CP_Radial_D8.0mm_P3.50mm
- C3: footprint Capacitor_SMD:C_1206_3216Metric_Pad1.33x1.80mm_HandSolder -> Capacitor_SMD:C_0603_1608Metric
- C6: value 100uF -> 220uF; footprint Capacitor_SMD:CP_Elec_10x10.5 -> Capacitor_THT:CP_Radial_D8.0mm_P3.50mm
- L1: value 10uh -> 4.7uH

Commit message: v0.41 done
Parts:
- added D8: SMF12A, Diode_SMD:D_SMF, symbol Diode:SMF12A
- D1: value SMAJ18A -> SMCJ18A
- R3, R4: value 4.7r -> 3.3R
- R6: value 274K -> 100K
- R7: value 274K -> 287K
- R9: value 274K -> 1K
Connections:
- net VOUT: now also D8.1 (A1); no longer R9.1
- new net: D8.2 (A2), R9.1
Changed lines of the file:
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@@
+    (stroke (width 0) (type default))
+  )
+  (wire (pts (xy 168.91 129.54) (xy 168.91 130.81))
     (stroke (width 0) (type default))
   )
@@
   )
   (wire (pts (xy 60.96 160.02) (xy 69.85 160.02))
+    (stroke (width 0) (type default))
+  )
+  (wire (pts (xy 168.91 118.11) (xy 168.91 121.92))
     (stroke (width 0) (type default))
   )
@@
     (effects (font (size 1.27 1.27)) (justify right))
   )
-  (hierarchical_label "VOUT" (shape input) (at 168.91 130.81 180) (fields_autoplaced)
+  (hierarchical_label "VOUT" (shape input) (at 168.91 118.11 180) (fields_autoplaced)
     (effects (font (size 1.27 1.27)) (justify right))
   )
@@
       (effects (font (size 1.27 1.27)) (justify left))
     )
-    (property "Value" "274K" (at 69.85 142.24 90)
+    (property "Value" "100K" (at 69.85 142.24 90)
       (effects (font (size 1.27 1.27)) (justify left))
     )
@@
       (effects (font (size 1.27 1.27)))
     )
-    (property "Value" "274K" (at 225.044 59.182 0)
+    (property "Value" "287K" (at 225.044 59.182 0)
       (effects (font (size 1.27 1.27)))
     )
@@
         (path "/e63e39d7-6ac0-4ffd-8aa3-1841a4541b55"
           (reference "R7") (unit 1)
+        )
+      )
+    )
+  )
+  (symbol (lib_id "Diode:SMF12A") (at 168.91 125.73 270) (unit 1)
+    (in_bom yes) (on_board yes) (dnp no) (fields_autoplaced)
+    (property "Reference" "D8" (at 171.45 125.095 90)
+      (effects (font (size 1.27 1.27)) (justify left))
+    )
+    (property "Value" "SMF12A" (at 171.45 127.635 90)
+      (effects (font (size 1.27 1.27)) (justify left))
+    )
+    (property "Footprint" "Diode_SMD:D_SMF" (at 163.83 125.73 0)
+      (effects (font (size 1.27 1.27)) hide)
+    )
+    (property "Datasheet" "https://www.vishay.com/doc?85881" (at 168.91 124.46 0)
+      (effects (font (size 1.27 1.27)) hide)
+    )
+    (pin "1")
+    (pin "2")
+    (instances
+      (project "24TO19_JYC_RM2023_V0.41_RY"
+        (path "/e63e39d7-6ac0-4ffd-8aa3-1841a4541b55"
+          (reference "D8") (unit 1)
         )
       )
@@
       (effects (font (size 1.27 1.27)) (justify right))
     )
-    (property "Value" "SMAJ18A" (at 50.8 154.94 90)
+    (property "Value" "SMCJ18A" (at 50.8 154.94 90)
       (effects (font (size 1.27 1.27)) (justify right))
     )
@@
       (effects (font (size 1.27 1.27)) (justify left))
     )
-    (property "Value" "274K" (at 171.45 136.525 0)
+    (property "Value" "1K" (at 171.45 136.525 0)
       (effects (font (size 1.27 1.27)) (justify left))
     )
@@
   (symbol (lib_id "Device:R") (at 162.56 45.72 90) (unit 1)
     (in_bom yes) (on_board yes) (dnp no) (fields_autoplaced)
-    (property "Reference" "R4" (at 162.56 39.116 90)
-      (effects (font (size 1.27 1.27)))
-    )
-    (property "Value" "4.7r" (at 162.56 41.656 90)
+    (property "Reference" "R4" (at 162.56 40.64 90)
+      (effects (font (size 1.27 1.27)))
+    )
+    (property "Value" "3.3R" (at 162.56 43.18 90)
       (effects (font (size 1.27 1.27)))
     )
@@
   (symbol (lib_id "Device:R") (at 162.56 68.58 90) (unit 1)
     (in_bom yes) (on_board yes) (dnp no) (fields_autoplaced)
-    (property "Reference" "R3" (at 162.56 61.976 90)
-      (effects (font (size 1.27 1.27)))
-    )
-    (property "Value" "4.7r" (at 162.56 64.516 90)
-      (effects (font (size 1.27 1.27)))
-    )
+    (property "Reference" "R3" (at 162.56 63.5 90)
+      (effects (font (size 1.27 1.27)))
+    )
+    (property "Value" "3.3R" (at 162.56 66.04 90)
+      (effects (font (size 1.27 1.27)))
+    )
